Commit message: update

File: Models/Frankenstein/new/FrankensteinV3.urdf (robot description, URDF)
Before this commit: robot panda, 62 links, 61 joints
Links:
- added link end_effector, mass 0; visual sphere radius=0.02
Joints:
- added joint aiming_joint: type fixed, parent panda_link8, child end_effector, origin xyz=0 0 0.12 rpy=0 0 0, axis 0 0 0

Commit message: first auto task working

File: Models/Frankenstein/new/FrankensteinV3.urdf (robot description, URDF)
Before this commit: robot panda, 63 links, 62 joints
Links:
- removed link base_tactile
Joints:
- removed joint base_tactile_joint
